Commit message: fixed stal files

File: so101_description/urdf/ignition.xacro (robot description, xacro)
@@ -1,3 +1,3 @@
-<!-- <?xml version="1.0"?>
+<?xml version="1.0"?>
 <robot xmlns:xacro="http://www.ros.org/wiki/xacro">
     <gazebo>
@@ -6,6 +6,6 @@
         </plugin>
     </gazebo>
-</robot> -->
-<?xml version="1.0"?>
+</robot>
+<!-- <?xml version="1.0"?>
 <robot xmlns:xacro="http://www.ros.org/wiki/xacro">
     <gazebo>
@@ -16,3 +16,3 @@
         </plugin>
     </gazebo>
-</robot>
+</robot> -->

File: so101_description/urdf/so101.urdf (robot description, URDF)
Before this commit: robot so101, 8 links, 7 joints
Links:
- removed link moving_jaw_so101_v1_link
- added link moving_jaw_so101_link, mass 0.012; collision mesh filename=package://so101_description/meshes/so101/moving_jaw_so101.s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; visual mesh filename=package://so101_description/meshes/so101/moving_jaw_so101.s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
- link base_link: geometry collision mesh filename=package://so101_description/meshes/so101/base_motor_holder_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; collision mesh filename=package://so101_description/meshes/so101/base_so101_v2.stl
- link gripper_link: geometry collision mesh filename=package://so101_description/meshes/so101/sts3215_03a.stl; collision mesh filename=package://so101_description/meshes/so101/wrist_roll_followe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
- link lower_arm_link: geometry collision mesh filename=package://so101_description/meshes/so101/motor_holder_so101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; collision mesh filename=package://so101_description/meshes/so101/sts3215_03a.stl
- link shoulder_link: geometry collision mesh filename=package://so101_description/meshes/so101/motor_holder_so101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; collision mesh filename=package://so101_description/meshes/so101/rotation_pitch_so1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
- link upper_arm_link: geometry collision mesh filename=package://so101_description/meshes/so101/sts3215_03a.stl; collision mesh filename=package://so101_description/meshes/so101/upper_arm_so101.stl
Joints:
- joint gripper: child moving_jaw_so101_v1_link -> moving_jaw_so101_link
