Commit message: added moveit and igntion sim is going on

File: so101_description/urdf/constants.xacro (robot description, xacro)
@@ -3,5 +3,5 @@
   <!-- Shared constants/properties (no includes here) -->
   <!-- <xacro:property name="mesh_dir" value="$(find so101_description)/meshes/assets"/> -->
-  <!-- <xacro:property name="mesh_dir" value="package://so101_description/meshes/so101"/> -->
+  <xacro:property name="MESH_DIR" value="package://so101_description/meshes/so101"/>
   <xacro:property name="default_effort"  value="10"/>
   <xacro:property name="default_velocity" value="10"/>

File: so101_description/urdf/joints.xacro (robot description, xacro)
@@ -1,8 +1,8 @@
 <?xml version="1.0"?>
 <robot xmlns:xacro="http://www.ros.org/wiki/xacro">
-  <joint name="world_to_base" type="fixed">
+  <!-- <joint name="world_to_base" type="fixed">
     <parent link="world"/>
     <child link="base_link"/>
-  </joint>
+  </joint> -->
   <!-- fixed: gripper_link -> gripper_frame_link -->
   <joint name="gripper_frame_joint" type="fixed">

File: so101_description/urdf/links.xacro (robot description, xacro)
@@ -1,5 +1,5 @@
 <?xml version="1.0"?>
 <robot xmlns:xacro="http://www.ros.org/wiki/xacro">
-  <link name="world"/>
+  <!-- <link name="world"/> -->
   <!-- Link base -->
   <link name="base_link">
@@ -13,5 +13,5 @@
       <origin xyz="-0.00636471 -9.94414e-05 -0.0024" rpy="1.5708 -1.67685e-15 1.5708"/>
       <geometry>
-        <mesh filename="package://so101_description/meshes/so101/base_motor_holder_so101_v1.stl"/>
+        <mesh filename="${MESH_DIR}/base_motor_holder_so101_v1.stl"/>
       </geometry>
       <material name="3d_printed"/>
@@ -20,5 +20,5 @@
       <origin xyz="-0.00636471 -9.94414e-05 -0.0024" rpy="1.5708 -1.67685e-15 1.5708"/>
       <geometry>
-        <mesh filename="package://so101_description/meshes/so101/base_motor_holder_so101_v1.stl"/>
+        <mesh filename="${MESH_DIR}/base_motor_holder_so101_v1.stl"/>
       </geometry>
     </collision>
@@ -27,5 +27,5 @@
       <origin xyz="-0.00636471 -8.97657e-09 -0.0024" rpy="1.5708 -2.78073e-29 1.5708"/>
       <geometry>
-        <mesh filename="package://so101_description/meshes/so101/base_so101_v2.stl"/>
+        <mesh filename="${MESH_DIR}/base_so101_v2.stl"/>
       </geometry>
       <material name="3d_printed"/>
@@ -34,5 +34,5 @@
       <origin xyz="-0.00636471 -8.97657e-09 -0.0024" rpy="1.5708 -2.78073e-29 1.5708"/>
       <geometry>
-        <mesh filename="package://so101_description/meshes/so101/base_so101_v2.stl"/>
+        <mesh filename="${MESH_DIR}/base_so101_v2.stl"/>
       </geometry>
     </collision>
@@ -41,5 +41,5 @@
       <origin xyz="0.0263353 -8.97657e-09 0.0437" rpy="-8.21148e-16 7.84513e-18 1.249e-15"/>
       <geometry>
-        <mesh filename="package://so101_description/meshes/so101/sts3215_03a_v1.stl"/>
+        <mesh filename="${MESH_DIR}/sts3215_03a_v1.stl"/>
       </geometry>
       <material name="sts3215"/>
@@ -48,5 +48,5 @@
       <origin xyz="0.0263353 -8.97657e-09 0.0437" rpy="-8.21148e-16 7.84513e-18 1.249e-15"/>
       <geometry>
-        <mesh filename="package://so101_description/meshes/so101/sts3215_03a_v1.stl"/>
+        <mesh filename="${MESH_DIR}/sts3215_03a_v1.stl"/>
       </geometry>
     </collision>
@@ -55,5 +55,5 @@
       <origin xyz="-0.0309827 -0.000199441 0.0474" rpy="1.5708 -1.35493e-14 1.5708"/>
       <geometry>
-        <mesh filename="package://so101_description/meshes/so101/waveshare_mounting_plate_so101_v2.stl"/>
+        <mesh filename="${MESH_DIR}/waveshare_mounting_plate_so101_v2.stl"/>
       </geometry>
       <material name="3d_printed"/>
@@ -62,5 +62,5 @@
       <origin xyz="-0.0309827 -0.000199441 0.0474" rpy="1.5708 -1.35493e-14 1.5708"/>
       <geometry>
-        <mesh filename="package://so101_description/meshes/so101/waveshare_mounting_plate_so101_v2.stl"/>
+        <mesh filename="${MESH_DIR}/waveshare_mounting_plate_so101_v2.stl"/>
       </geometry>
     </collision>
@@ -77,5 +77,5 @@
       <origin xyz="-0.0303992 0.000422241 -0.0417" rpy="1.5708 1.5708 0"/>
       <geometry>
-        <mesh filename="package://so101_description/meshes/so101/sts3215_03a_v1.stl"/>
+        <mesh filename="${MESH_DIR}/sts3215_03a_v1.stl"/>
       </geometry>
       <material name="sts3215"/>
@@ -84,5 +84,5 @@
       <origin xyz="-0.0303992 0.000422241 -0.0417" rpy="1.5708 1.5708 0"/>
       <geometry>
-        <mesh filename="package://so101_description/meshes/so101/sts3215_03a_v1.stl"/>
+        <mesh filename="${MESH_DIR}/sts3215_03a_v1.stl"/>
       </geometry>
     </collision>
@@ -91,5 +91,5 @@
       <origin xyz="-0.0675992 -0.000177759 0.0158499" rpy="1.5708 -1.5708 0"/>
       <geometry>
-        <mesh filename="package://so101_description/meshes/so101/motor_holder_so101_base_v1.stl"/>
+        <mesh filename="${MESH_DIR}/motor_holder_so101_base_v1.stl"/>
       </geometry>
       <material name="3d_printed"/>
@@ -98,5 +98,5 @@
       <origin xyz="-0.0675992 -0.000177759 0.0158499" rpy="1.5708 -1.5708 0"/>
       <geometry>
-        <mesh filename="package://so101_description/meshes/so101/motor_holder_so101_base_v1.stl"/>
+        <mesh filename="${MESH_DIR}/motor_holder_so101_base_v1.stl"/>
       </geometry>
     </collision>
@@ -105,5 +105,5 @@
       <origin xyz="0.0122008 2.22413e-05 0.0464" rpy="-1.5708 2.35221e-33 0"/>
       <geometry>
-        <mesh filename="package://so101_description/meshes/so101/rotation_pitch_so101_v1.stl"/>
+        <mesh filename="${MESH_DIR}/rotation_pitch_so101_v1.stl"/>
       </geometry>
       <material name="3d_printed"/>
@@ -112,5 +112,5 @@
       <origin xyz="0.0122008 2.22413e-05 0.0464" rpy="-1.5708 2.35221e-33 0"/>
       <geometry>
-        <mesh filename="package://so101_description/meshes/so101/rotation_pitch_so101_v1.stl"/>
+        <mesh filename="${MESH_DIR}/rotation_pitch_so101_v1.stl"/>
       </geometry>
     </collision>
@@ -127,5 +127,5 @@
       <origin xyz="-0.11257 -0.0155 0.0187" rpy="-3.14159 -5.27356e-16 -1.5708"/>
       <geometry>
-        <mesh filename="package://so101_description/meshes/so101/sts3215_03a_v1.stl"/>
+        <mesh filename="${MESH_DIR}/sts3215_03a_v1.stl"/>
       </geometry>
       <material name="sts3215"/>
@@ -134,5 +134,5 @@
       <origin xyz="-0.11257 -0.0155 0.0187" rpy="-3.14159 -5.27356e-16 -1.5708"/>
       <geometry>
-        <mesh filename="package://so101_description/meshes/so101/sts3215_03a_v1.stl"/>
+        <mesh filename="${MESH_DIR}/sts3215_03a_v1.stl"/>
       </geometry>
     </collision>
@@ -141,5 +141,5 @@
       <origin xyz="-0.065085 0.012 0.0182" rpy="3.14159 -0 -1.30911e-30"/>
       <geometry>
-        <mesh filename="package://so101_description/meshes/so101/upper_arm_so101_v1.stl"/>
+        <mesh filename="${MESH_DIR}/upper_arm_so101_v1.stl"/>
       </geometry>
       <material name="3d_printed"/>
@@ -148,5 +148,5 @@
       <origin xyz="-0.065085 0.012 0.0182" rpy="3.14159 -0 -1.30911e-30"/>
       <geometry>
-        <mesh filename="package://so101_description/meshes/so101/upper_arm_so101_v1.stl"/>
+        <mesh filename="${MESH_DIR}/upper_arm_so101_v1.stl"/>
       </geometry>
     </collision>
@@ -163,5 +163,5 @@
       <origin xyz="-0.0648499 -0.032 0.0182" rpy="3.14159 -0 6.67202e-31"/>
       <geometry>
-        <mesh filename="package://so101_description/meshes/so101/under_arm_so101_v1.stl"/>
+        <mesh filename="${MESH_DIR}/under_arm_so101_v1.stl"/>
       </geometry>
       <material name="3d_printed"/>
@@ -170,5 +170,5 @@
       <origin xyz="-0.0648499 -0.032 0.0182" rpy="3.14159 -0 6.67202e-31"/>
       <geometry>
-        <mesh filename="package://so101_description/meshes/so101/under_arm_so101_v1.stl"/>
+        <mesh filename="${MESH_DIR}/under_arm_so101_v1.stl"/>
       </geometry>
     </collision>
@@ -177,5 +177,5 @@
       <origin xyz="-0.0648499 -0.032 0.018" rpy="-3.14159 -2.55351e-15 -1.83387e-30"/>
       <geometry>
-        <mesh filename="package://so101_description/meshes/so101/motor_holder_so101_wrist_v1.stl"/>
+        <mesh filename="${MESH_DIR}/motor_holder_so101_wrist_v1.stl"/>
       </geometry>
       <material name="3d_printed"/>
@@ -184,5 +184,5 @@
       <origin xyz="-0.0648499 -0.032 0.018" rpy="-3.14159 -2.55351e-15 -1.83387e-30"/>
       <geometry>
-        <mesh filename="package://so101_description/meshes/so101/motor_holder_so101_wrist_v1.stl"/>
+        <mesh filename="${MESH_DIR}/motor_holder_so101_wrist_v1.stl"/>
       </geometry>
     </collision>
@@ -191,5 +191,5 @@
       <origin xyz="-0.1224 0.0052 0.0187" rpy="-3.14159 -7.88861e-31 -3.14159"/>
       <geometry>
-        <mesh filename="package://so101_description/meshes/so101/sts3215_03a_v1.stl"/>
+        <mesh filename="${MESH_DIR}/sts3215_03a_v1.stl"/>
       </geometry>
       <material name="sts3215"/>
@@ -198,5 +198,5 @@
       <origin xyz="-0.1224 0.0052 0.0187" rpy="-3.14159 -7.88861e-31 -3.14159"/>
       <geometry>
-        <mesh filename="package://so101_description/meshes/so101/sts3215_03a_v1.stl"/>
+        <mesh filename="${MESH_DIR}/sts3215_03a_v1.stl"/>
       </geometry>
     </collision>
@@ -213,5 +213,5 @@
       <origin xyz="8.32667e-17 -0.0424 0.0306" rpy="1.5708 1.5708 0"/>
       <geometry>
-        <mesh filename="package://so101_description/meshes/so101/sts3215_03a_no_horn_v1.stl"/>
+        <mesh filename="${MESH_DIR}/sts3215_03a_no_horn_v1.stl"/>
       </geometry>
       <material name="sts3215"/>
@@ -220,5 +220,5 @@
       <origin xyz="8.32667e-17 -0.0424 0.0306" rpy="1.5708 1.5708 0"/>
       <geometry>
-        <mesh filename="package://so101_description/meshes/so101/sts3215_03a_no_horn_v1.stl"/>
+        <mesh filename="${MESH_DIR}/sts3215_03a_no_horn_v1.stl"/>
       </geometry>
     </collision>
@@ -227,5 +227,5 @@
       <origin xyz="0 -0.028 0.0181" rpy="-1.5708 -1.5708 0"/>
       <geometry>
-        <mesh filename="package://so101_description/meshes/so101/wrist_roll_pitch_so101_v2.stl"/>
+        <mesh filename="${MESH_DIR}/wrist_roll_pitch_so101_v2.stl"/>
       </geometry>
       <material name="3d_printed"/>
@@ -234,5 +234,5 @@
       <origin xyz="0 -0.028 0.0181" rpy="-1.5708 -1.5708 0"/>
       <geometry>
-        <mesh filename="package://so101_description/meshes/so101/wrist_roll_pitch_so101_v2.stl"/>
+        <mesh filename="${MESH_DIR}/wrist_roll_pitch_so101_v2.stl"/>
       </geometry>
     </collision>
@@ -249,5 +249,5 @@
       <origin xyz="0.0077 0.0001 -0.0234" rpy="-1.5708 -5.19179e-17 -1.66533e-16"/>
       <geometry>
-        <mesh filename="package://so101_description/meshes/so101/sts3215_03a_v1.stl"/>
+        <mesh filename="${MESH_DIR}/sts3215_03a_v1.stl"/>
       </geometry>
       <material name="sts3215"/>
@@ -256,5 +256,5 @@
       <origin xyz="0.0077 0.0001 -0.0234" rpy="-1.5708 -5.19179e-17 -1.66533e-16"/>
       <geometry>
-        <mesh filename="package://so101_description/meshes/so101/sts3215_03a_v1.stl"/>
+        <mesh filename="${MESH_DIR}/sts3215_03a_v1.stl"/>
       </geometry>
     </collision>
@@ -263,5 +263,5 @@
       <origin xyz="8.32667e-17 -0.000218214 0.000949706" rpy="-3.14159 -5.55112e-17 0"/>
       <geometry>
-        <mesh filename="package://so101_description/meshes/so101/wrist_roll_follower_so101_v1.stl"/>
+        <mesh filename="${MESH_DIR}/wrist_roll_follower_so101_v1.stl"/>
       </geometry>
       <material name="3d_printed"/>
@@ -270,5 +270,5 @@
       <origin xyz="8.32667e-17 -0.000218214 0.000949706" rpy="-3.14159 -5.55112e-17 0"/>
       <geometry>
-        <mesh filename="package://so101_description/meshes/so101/wrist_roll_follower_so101_v1.stl"/>
+        <mesh filename="${MESH_DIR}/wrist_roll_follower_so101_v1.stl"/>
       </geometry>
     </collision>
@@ -294,5 +294,5 @@
       <origin xyz="-5.55112e-17 -5.55112e-17 0.0189" rpy="9.53145e-17 6.93889e-18 1.24077e-24"/>
       <geometry>
-        <mesh filename="package://so101_description/meshes/so101/moving_jaw_so101_v1.stl"/>
+        <mesh filename="${MESH_DIR}/moving_jaw_so101_v1.stl"/>
       </geometry>
       <material name="3d_printed"/>
@@ -301,5 +301,5 @@
       <origin xyz="-5.55112e-17 -5.55112e-17 0.0189" rpy="9.53145e-17 6.93889e-18 1.24077e-24"/>
       <geometry>
-        <mesh filename="package://so101_description/meshes/so101/moving_jaw_so101_v1.stl"/>
+        <mesh filename="${MESH_DIR}/moving_jaw_so101_v1.stl"/>
       </geometry>
     </collision>

File: so101_description/urdf/ros2_control.xacro (robot description, xacro)
@@ -1,46 +1,45 @@
 <?xml version="1.0"?>
 <robot xmlns:xacro="http://www.ros.org/wiki/xacro">
-  <xacro:macro name="so101_ros2_control">
-    <ros2_control name="so101_hw" type="system">
-        <hardware>
-            <plugin>mock_components/GenericSystem</plugin>
-            <param name="calculate_dynamics">false</param>
-            <param name="custom_interface_with_following_offset"></param>
-            <param name="disable_commands">false</param>
-            <param name="mock_gpio_commands">false</param>
-            <param name="mock_sensor_commands">false</param>
-            <param name="position_state_following_offset">0.0</param>
-        </hardware>
-        <joint name="shoulder_pan">
-        <command_interface name="position"/>
-        <state_interface   name="position"/>
-        <state_interface   name="velocity"/>
-        </joint>
-        <joint name="shoulder_lift">
-        <command_interface name="position"/>
-        <state_interface   name="position"/>
-        <state_interface   name="velocity"/>
-        </joint>
-        <joint name="elbow_flex">
-        <command_interface name="position"/>
-        <state_interface   name="position"/>
-        <state_interface   name="velocity"/>
-        </joint>
-        <joint name="wrist_flex">
-        <command_interface name="position"/>
-        <state_interface   name="position"/>
-        <state_interface   name="velocity"/>
-        </joint>
-        <joint name="wrist_roll">
-        <command_interface name="position"/>
-        <state_interface   name="position"/>
-        <state_interface   name="velocity"/>
-        </joint>
-        <joint name="gripper">
-        <command_interface name="position"/>
-        <state_interface   name="position"/>
-        <state_interface   name="velocity"/>
-        </joint>
-    </ros2_control>
-  </xacro:macro>
+  <ros2_control name="so101_hw" type="system">
+    <hardware>
+      <!-- <plugin>mock_components/GenericSystem</plugin>
+      <param name="calculate_dynamics">false</param>
+      <param name="custom_interface_with_following_offset"></param>
+      <param name="disable_commands">false</param>
+      <param name="mock_gpio_commands">false</param>
+      <param name="mock_sensor_commands">false</param>
+      <param name="position_state_following_offset">0.0</param> -->
+      <plugin>ign_ros2_control/IgnitionSystem</plugin>
+    </hardware>
+    <joint name="shoulder_pan">
+      <command_interface name="position"/>
+      <state_interface   name="position"/>
+      <state_interface   name="velocity"/>
+    </joint>
+    <joint name="shoulder_lift">
+      <command_interface name="position"/>
+      <state_interface   name="position"/>
+      <state_interface   name="velocity"/>
+    </joint>
+    <joint name="elbow_flex">
+      <command_interface name="position"/>
+      <state_interface   name="position"/>
+      <state_interface   name="velocity"/>
+    </joint>
+    <joint name="wrist_flex">
+      <command_interface name="position"/>
+      <state_interface   name="position"/>
+      <state_interface   name="velocity"/>
+    </joint>
+    <joint name="wrist_roll">
+      <command_interface name="position"/>
+      <state_interface   name="position"/>
+      <state_interface   name="velocity"/>
+    </joint>
+    <joint name="gripper">
+      <command_interface name="position"/>
+      <state_interface   name="position"/>
+      <state_interface   name="velocity"/>
+    </joint>
+  </ros2_control>
 </robot>

File: so101_description/urdf/so101.urdf (robot description, URDF)
Before this commit: robot so101, 9 links, 8 joints
Links:
- removed link world
Joints:
- removed joint world_to_base

File: so101_description/urdf/so101.urdf.xacro (robot description, xacro)
@@ -9,3 +9,4 @@
   <!-- For ROS 2 control (optional; add when you wire controllers) -->
   <xacro:include filename="$(find so101_description)/urdf/ros2_control.xacro"/>
+  <xacro:include filename="$(find so101_description)/urdf/ignition.xacro"/>
 </robot>
