Commit message: modified urdf added condiitons

File: so101_description/urdf/constants.xacro (robot description, xacro)
@@ -6,17 +6,9 @@
   <xacro:property name="default_effort"  value="10"/>
   <xacro:property name="default_velocity" value="10"/>
-  <!-- STL filenames (as used by your original file) -->
-  <!-- <xacro:property name="stl_base_holder"           value="base_motor_holder_so101_v1.stl"/>
-  <xacro:property name="stl_base"                  value="base_so101_v2.stl"/>
-  <xacro:property name="stl_servo"                 value="sts3215_03a_v1.stl"/>
-  <xacro:property name="stl_servo_nohorn"          value="sts3215_03a_no_horn_v1.stl"/>
-  <xacro:property name="stl_waveshare"             value="waveshare_mounting_plate_so101_v2.stl"/>
-  <xacro:property name="stl_rotation_pitch"        value="rotation_pitch_so101_v1.stl"/>
-  <xacro:property name="stl_upper_arm"             value="upper_arm_so101_v1.stl"/>
-  <xacro:property name="stl_under_arm"             value="under_arm_so101_v1.stl"/>
-  <xacro:property name="stl_wrist_holder"          value="motor_holder_so101_wrist_v1.stl"/>
-  <xacro:property name="stl_wrist_roll_pitch"      value="wrist_roll_pitch_so101_v2.stl"/>
-  <xacro:property name="stl_wrist_roll_follower"   value="wrist_roll_follower_so101_v1.stl"/>
-  <xacro:property name="stl_moving_jaw"            value="moving_jaw_so101_v1.stl"/>
-  <xacro:property name="stl_motor_holder_base"     value="motor_holder_so101_base_v1.stl"/> -->
+  <!-- Define arguments with default values -->
+  <xacro:arg name="use_ros2_control" default="true"/>
+  <xacro:arg name="use_ignition" default="true"/>
+  <!-- Convert arguments to properties for use in included files -->
+  <xacro:property name="use_ros2_control" value="$(arg use_ros2_control)"/>
+  <xacro:property name="use_ignition" value="$(arg use_ignition)"/>
 </robot>

File: so101_description/urdf/ignition.xacro (robot description, xacro)
@@ -1,3 +1,16 @@
 <?xml version="1.0"?>
+<robot xmlns:xacro="http://www.ros.org/wiki/xacro">
+    <!-- Define a property that can be set at xacro command -->
+    <xacro:if value="${use_ignition}">
+        <gazebo>
+            <plugin filename="libign_ros2_control-system.so" name="ign_ros2_control::IgnitionROS2ControlPlugin">
+                <parameters>$(find so101_bringup)/config/so101_controllers.yaml</parameters>
+                <robot_param>robot_description</robot_param>
+                <robot_param_node>robot_state_publisher</robot_param_node>
+            </plugin>
+        </gazebo>
+    </xacro:if>
+</robot>
+<!-- <?xml version="1.0"?>
 <robot xmlns:xacro="http://www.ros.org/wiki/xacro">
     <gazebo>
@@ -6,13 +19,3 @@
         </plugin>
     </gazebo>
-</robot>
-<!-- <?xml version="1.0"?>
-<robot xmlns:xacro="http://www.ros.org/wiki/xacro">
-    <gazebo>
-        <plugin filename="libign_ros2_control-system.so" name="ign_ros2_control::IgnitionROS2ControlPlugin">
-            <parameters>$(find so101_bringup)/config/so101_controllers.yaml</parameters>
-            <robot_param>robot_description</robot_param>
-            <robot_param_node>robot_state_publisher</robot_param_node>
-        </plugin>
-    </gazebo>
 </robot> -->

File: so101_description/urdf/ros2_control.xacro (robot description, xacro)
@@ -1,45 +1,51 @@
 <?xml version="1.0"?>
 <robot xmlns:xacro="http://www.ros.org/wiki/xacro">
-  <ros2_control name="so101_hw" type="system">
-    <hardware>
-      <!-- <plugin>mock_components/GenericSystem</plugin>
-      <param name="calculate_dynamics">false</param>
-      <param name="custom_interface_with_following_offset"></param>
-      <param name="disable_commands">false</param>
-      <param name="mock_gpio_commands">false</param>
-      <param name="mock_sensor_commands">false</param>
-      <param name="position_state_following_offset">0.0</param> -->
-      <plugin>ign_ros2_control/IgnitionSystem</plugin>
-    </hardware>
-    <joint name="shoulder_pan">
-      <command_interface name="position"/>
-      <state_interface   name="position"/>
-      <state_interface   name="velocity"/>
-    </joint>
-    <joint name="shoulder_lift">
-      <command_interface name="position"/>
-      <state_interface   name="position"/>
-      <state_interface   name="velocity"/>
-    </joint>
-    <joint name="elbow_flex">
-      <command_interface name="position"/>
-      <state_interface   name="position"/>
-      <state_interface   name="velocity"/>
-    </joint>
-    <joint name="wrist_flex">
-      <command_interface name="position"/>
-      <state_interface   name="position"/>
-      <state_interface   name="velocity"/>
-    </joint>
-    <joint name="wrist_roll">
-      <command_interface name="position"/>
-      <state_interface   name="position"/>
-      <state_interface   name="velocity"/>
-    </joint>
-    <joint name="gripper">
-      <command_interface name="position"/>
-      <state_interface   name="position"/>
-      <state_interface   name="velocity"/>
-    </joint>
-  </ros2_control>
+  <xacro:if value="${use_ros2_control}">
+    <ros2_control name="so101_hw" type="system">
+      <hardware>
+        <xacro:if value="${use_ignition}">
+          <plugin>ign_ros2_control/IgnitionSystem</plugin>
+        </xacro:if>
+        <xacro:unless value="${use_ignition}">
+          <plugin>mock_components/GenericSystem</plugin>
+          <param name="calculate_dynamics">false</param>
+          <param name="custom_interface_with_following_offset"></param>
+          <param name="disable_commands">false</param>
+          <param name="mock_gpio_commands">false</param>
+          <param name="mock_sensor_commands">false</param>
+          <param name="position_state_following_offset">0.0</param>
+        </xacro:unless>
+      </hardware>
+      <joint name="shoulder_pan">
+        <command_interface name="position"/>
+        <state_interface   name="position"/>
+        <state_interface   name="velocity"/>
+      </joint>
+      <joint name="shoulder_lift">
+        <command_interface name="position"/>
+        <state_interface   name="position"/>
+        <state_interface   name="velocity"/>
+      </joint>
+      <joint name="elbow_flex">
+        <command_interface name="position"/>
+        <state_interface   name="position"/>
+        <state_interface   name="velocity"/>
+      </joint>
+      <joint name="wrist_flex">
+        <command_interface name="position"/>
+        <state_interface   name="position"/>
+        <state_interface   name="velocity"/>
+      </joint>
+      <joint name="wrist_roll">
+        <command_interface name="position"/>
+        <state_interface   name="position"/>
+        <state_interface   name="velocity"/>
+      </joint>
+      <joint name="gripper">
+        <command_interface name="position"/>
+        <state_interface   name="position"/>
+        <state_interface   name="velocity"/>
+      </joint>
+    </ros2_control>
+  </xacro:if>
 </robot>

Commit message: simulaiton all set

File: so101_description/urdf/constants.xacro (robot description, xacro)
@@ -9,6 +9,8 @@
   <xacro:arg name="use_ros2_control" default="true"/>
   <xacro:arg name="use_ignition" default="true"/>
+  <xacro:arg name="use_hardware" default="false"/>
   <!-- Convert arguments to properties for use in included files -->
   <xacro:property name="use_ros2_control" value="$(arg use_ros2_control)"/>
   <xacro:property name="use_ignition" value="$(arg use_ignition)"/>
+  <xacro:property name="use_hardware" value="$(arg use_hardware)"/>
 </robot>

File: so101_description/urdf/joints.xacro (robot description, xacro)
@@ -1,8 +1,8 @@
 <?xml version="1.0"?>
 <robot xmlns:xacro="http://www.ros.org/wiki/xacro">
-  <!-- <joint name="world_to_base" type="fixed">
+  <joint name="world_to_base" type="fixed">
     <parent link="world"/>
     <child link="base_link"/>
-  </joint> -->
+  </joint>
   <!-- fixed: gripper_link -> gripper_frame_link -->
   <joint name="gripper_frame_joint" type="fixed">

File: so101_description/urdf/links.xacro (robot description, xacro)
@@ -1,5 +1,5 @@
 <?xml version="1.0"?>
 <robot xmlns:xacro="http://www.ros.org/wiki/xacro">
-  <!-- <link name="world"/> -->
+  <link name="world"/>
   <!-- Link base -->
   <link name="base_link">

File: so101_description/urdf/ros2_control.xacro (robot description, xacro)
@@ -4,19 +4,25 @@
     <ros2_control name="so101_hw" type="system">
       <hardware>
+        <!-- Case 1: Ignition/Gazebo simulation -->
         <xacro:if value="${use_ignition}">
           <plugin>ign_ros2_control/IgnitionSystem</plugin>
         </xacro:if>
+        <!-- Case 2: Real hardware -->
         <xacro:unless value="${use_ignition}">
-          <plugin>mock_components/GenericSystem</plugin>
-          <param name="calculate_dynamics">false</param>
-          <param name="custom_interface_with_following_offset"></param>
-          <param name="disable_commands">false</param>
-          <param name="mock_gpio_commands">false</param>
-          <param name="mock_sensor_commands">false</param>
-          <param name="position_state_following_offset">0.0</param>
+          <xacro:if value="${use_hardware}">
+            <plugin>so101_hardware/So101System</plugin>
+            <param name="port">/dev/ttyUSB0</param>
+            <param name="baud_rate">115200</param>
+          </xacro:if>
+          <!-- Case 3: Mock/fake system (default if not ignition, not hardware) -->
+          <xacro:unless value="${use_hardware}">
+            <plugin>mock_components/GenericSystem</plugin>
+            <param name="calculate_dynamics">false</param>
+            <param name="disable_commands">false</param>
+            <param name="mock_gpio_commands">false</param>
+            <param name="mock_sensor_commands">false</param>
+            <param name="position_state_following_offset">0.0</param>
+          </xacro:unless>
         </xacro:unless>
-        <!-- <hardware>
-          <plugin>gz_ros2_control/GazeboSimSystem</plugin>
-        </hardware> -->
       </hardware>
       <joint name="shoulder_pan">
